Commit message: real_limo

File: src/limo_cobot_sim/limo_mycobot/limo/limo_description/urdf/limo_four_diff.xacro (robot description, xacro)
@@ -4,175 +4,10 @@
   <xacro:arg name="robot_namespace" default="/" />
   <xacro:arg name="frame_prefix" default="limo" />
-    <!-- <xacro:property name="frame_prefix" value="${frame_prefix}"/>
-    <xacro:property name="robot_namespace" value="${robot_namespace}"/> -->
   <xacro:include filename="$(find limo_description)/urdf/limo_xacro.xacro" />
-  <!-- <xacro:include filename="$(find limo_description)/urdf/limo_four_diff.gazebo" /> -->
-  <!-- <xacro:include filename="$(find limo_description)/urdf/limo_four_diff.gazebo"/> -->
-<xacro:property name="frame_prefix" value="$(arg frame_prefix)"/>
-<xacro:property name="robot_namespace" value="$(arg robot_namespace)"/>
-<xacro:macro name="limo_wheel_transmission" params="wheel_prefix">
-    <transmission name="${frame_prefix}_${wheel_prefix}_wheel_trans" type="SimpleTransmission">
-      <type>transmission_interface/SimpleTransmission</type>
-      <actuator name="${frame_prefix}_${wheel_prefix}_wheel_motor">
-        <hardwareInterface>hardware_interface/VelocityJointInterface</hardwareInterface>
-        <mechanicalReduction>1</mechanicalReduction>
-      </actuator>
-      <joint name="${frame_prefix}_${wheel_prefix}_wheel">
-        <hardwareInterface>hardware_interface/VelocityJointInterface</hardwareInterface>
-      </joint>
-    </transmission>
-  </xacro:macro>
-  <xacro:macro name="limo_steering_hinge_transmission" params="wheel_prefix">
-    <transmission name="${frame_prefix}_${wheel_prefix}_wheel_trans" type="SimpleTransmission">
-      <type>transmission_interface/SimpleTransmission</type>
-      <actuator name="${frame_prefix}_${wheel_prefix}_wheel_motor">
-        <hardwareInterface>hardware_interface/EffortJointInterface</hardwareInterface>
-        <mechanicalReduction>1</mechanicalReduction>
-      </actuator>
-      <joint name="${frame_prefix}_${wheel_prefix}_wheel">
-        <hardwareInterface>hardware_interface/EffortJointInterface</hardwareInterface>
-      </joint>
-    </transmission>
-  </xacro:macro>
-  <!-- Laser Macro -->
-  <xacro:macro name="gazebo_laser" params="frame_prefix">
-    <gazebo reference="${frame_prefix}_link">
-      <sensor type="ray" name="${frame_prefix}_laser_sensor">
-        <pose>0 0 0 0 0 0</pose>
-        <visualize>false</visualize>
-        <update_rate>8</update_rate>
-        <ray>
-          <scan>
-            <horizontal>
-              <samples>720</samples>
-              <resolution>1</resolution>
-              <min_angle>-2.09439504</min_angle>
-              <max_angle>2.09439504</max_angle>
-            </horizontal>
-          </scan>
-          <range>
-            <min>0.05</min>
-            <max>8.0</max>
-            <resolution>0.01</resolution>
-          </range>
-          <noise>
-            <type>gaussian</type>
-            <mean>0.0</mean>
-            <stddev>0.01</stddev>
-          </noise>
-        </ray>
-        <plugin name="${frame_prefix}_laser_plugin" filename="libgazebo_ros_laser.so">
-          <topicName>${robot_namespace}/scan</topicName>
-          <frameName>${frame_prefix}_link</frameName>
-        </plugin>
-      </sensor>
-    </gazebo>
-  </xacro:macro>
-  <!-- Depth Camera Macro -->
-  <xacro:macro name="gazebo_depth_camera" params="frame_prefix">
-    <gazebo reference="${frame_prefix}_link">
-      <sensor name="${frame_prefix}_depth_camera_sensor" type="depth">
-        <pose>0.0 0.0 0.0 0.0 0.0 0.0</pose>
-        <always_on>true</always_on>
-        <visualize>true</visualize>
-        <update_rate>10.0</update_rate>
-        <camera name="head">
-          <horizontal_fov>1.3962634</horizontal_fov>
-          <image>
-            <width>640</width>
-            <height>480</height>
-            <format>R8G8B8</format>
-          </image>
-          <clip>
-            <near>0.02</near>
-            <far>300</far>
-          </clip>
-        </camera>
-        <plugin name="${frame_prefix}_depth_camera_plugin" filename="libgazebo_ros_openni_kinect.so">
-          <baseline>0.2</baseline>
-          <alwaysOn>true</alwaysOn>
-          <updateRate>0.0</updateRate>
-          <cameraName>camera_ir</cameraName>
-          <imageTopicName>${robot_namespace}/color/image_raw</imageTopicName>
-          <cameraInfoTopicName>${robot_namespace}/color/camera_info</cameraInfoTopicName>
-          <depthImageTopicName>${robot_namespace}/depth/image_raw</depthImageTopicName>
-          <depthImageCameraInfoTopicName>${robot_namespace}/depth/camera_info</depthImageCameraInfoTopicName>
-          <pointCloudTopicName>${robot_namespace}/depth/points</pointCloudTopicName>
-          <frameName>${frame_prefix}_depth_link</frameName>
-          <cameraname>${frame_prefix}_depth_camera_link</cameraname>
-          <pointCloudCutoff>0.5</pointCloudCutoff>
-          <pointCloudCutoffMax>3.0</pointCloudCutoffMax>
-        </plugin>
-      </sensor>
-    </gazebo>
-  </xacro:macro>
-  <!-- IMU Macro -->
-  <xacro:macro name="gazebo_imu" params="frame_prefix">
-    <gazebo reference="${frame_prefix}_link">
-      <gravity>true</gravity>
-      <sensor name="${frame_prefix}_imu_sensor" type="imu">
-        <always_on>true</always_on>
-        <update_rate>100</update_rate>
-        <visualize>true</visualize>
-        <topic>__default_topic__</topic>
-        <plugin filename="libgazebo_ros_imu_sensor.so" name="${frame_prefix}_imu_plugin">
-          <topicName>${robot_namespace}/imu</topicName>
-          <bodyName>${frame_prefix}_link</bodyName>
-          <updateRateHZ>100.0</updateRateHZ>
-          <gaussianNoise>0.001</gaussianNoise>
-          <xyzOffset>0 0 0</xyzOffset>
-          <rpyOffset>0 0 0</rpyOffset>
-          <frameName>${frame_prefix}_imu_link</frameName>
-        </plugin>
-        <pose>0 0 0 0 0 0</pose>
-      </sensor>
-    </gazebo>
-  </xacro:macro>
-    <!-- Sensors -->
-    <xacro:gazebo_laser frame_prefix="${frame_prefix}_laser" />
-    <xacro:gazebo_depth_camera frame_prefix="${frame_prefix}_depth_camera" />
-    <xacro:gazebo_imu frame_prefix="${frame_prefix}_imu" />
-    <!-- Wheel contact parameters -->
-    <gazebo reference="${frame_prefix}_front_left_wheel">
-        <mu1>10</mu1><mu2>10</mu2><kp>10000000.0</kp><kd>1.0</kd>
-        <minDepth>0.01</minDepth><fdir1>1 0 0</fdir1><maxContacts value="64"/>
-    </gazebo>
-    <gazebo reference="${frame_prefix}_front_right_wheel">
-        <mu1>10</mu1><mu2>10</mu2><kp>10000000.0</kp><kd>1.0</kd>
-        <minDepth>0.01</minDepth><fdir1>1 0 0</fdir1><maxContacts value="64"/>
-    </gazebo>
-    <gazebo reference="${frame_prefix}_rear_left_wheel">
-        <mu1>10</mu1><mu2>10</mu2><kp>10000000.0</kp><kd>1.0</kd>
-        <minDepth>0.01</minDepth><fdir1>1 0 0</fdir1><maxContacts value="64"/>
-    </gazebo>
-    <gazebo reference="${frame_prefix}_rear_right_wheel">
-        <mu1>10</mu1><mu2>10</mu2><kp>10000000.0</kp><kd>1.0</kd>
-        <minDepth>0.01</minDepth><fdir1>1 0 0</fdir1><maxContacts value="64"/>
-    </gazebo>
-    <!-- Skid-steer drive plugin -->
-    <gazebo>
-        <plugin name="four_diff_controller" filename="libgazebo_ros_skid_steer_drive.so">
-            <updateRate>100.0</updateRate>
-            <robotNamespace>/${robot_namespace}</robotNamespace>
-            <leftFrontJoint>${frame_prefix}_front_left_wheel</leftFrontJoint>
-            <rightFrontJoint>${frame_prefix}_front_right_wheel</rightFrontJoint>
-            <leftRearJoint>${frame_prefix}_rear_left_wheel</leftRearJoint>
-            <rightRearJoint>${frame_prefix}_rear_right_wheel</rightRearJoint>
-            <wheelSeparation>0.172</wheelSeparation>
-            <wheelDiameter>0.09</wheelDiameter>
-            <robotBaseFrame>${frame_prefix}_base_footprint</robotBaseFrame>
-            <commandTopic>/${robot_namespace}/cmd_vel</commandTopic>
-            <torque>50</torque>
-            <broadcastTF>true</broadcastTF>
-            <odometryTopic>/${robot_namespace}/odom</odometryTopic>
-            <odometryFrame>${frame_prefix}_odom</odometryFrame>
-            <covariance_x>0.000100</covariance_x>
-            <covariance_y>0.000100</covariance_y>
-            <covariance_yaw>0.010000</covariance_yaw>
-        </plugin>
-    </gazebo>
+  <xacro:property name="frame_prefix" value="$(arg frame_prefix)"/>
+  <xacro:property name="robot_namespace" value="$(arg robot_namespace)"/>
   <!-- Variables -->
   <xacro:property name="M_PI" value="3.14159"/>
-  <!-- Vehicle Geometries -->
+  <!-- Simplified Vehicle Geometries -->
   <xacro:property name="base_x_size" value="0.13" />
   <xacro:property name="base_y_size" value="0.12" />
@@ -184,5 +19,5 @@
   <xacro:property name="wheel_length" value="0.045" />
   <xacro:property name="wheel_radius" value="0.045" />
-  <!-- Prefixed links/joints to avoid collisions when spawning multiple robots -->
+  <!-- Prefixed links/joints -->
   <link name="${frame_prefix}_base_footprint"/>
   <joint name="${frame_prefix}_base_joint" type="fixed">
@@ -191,20 +26,21 @@
     <origin xyz="0.0 0.0 0.15" rpy="0 0 0"/>
   </joint>
-  <!-- Base link -->
+  <!-- Simplified Base link - using box geometry instead of mesh -->
   <link name="${frame_prefix}_base_link">
       <visual>
-          <origin xyz="0 0 -0.15" rpy="0 0 1.57" />
+          <origin xyz="0 0 0" rpy="0 0 0" />
           <geometry>
-              <mesh filename="package://limo_description/meshes/limo_base.dae" scale="1 1 1"/>
+              <box size="${base_x_size} ${base_y_size} ${base_z_size}"/>
           </geometry>
+          <material name="grey">
+              <color rgba="0.5 0.5 0.5 1.0"/>
+          </material>
       </visual>
       <collision>
           <origin xyz="0 0 0" rpy="0 0 0" />
-        <geometry>
-            <box size="${base_x_size} ${base_y_size} ${base_z_size}"/>
-        </geometry>
+          <geometry>
+              <box size="${base_x_size} ${base_y_size} ${base_z_size}"/>
+          </geometry>
       </collision>
-  </link>
-  <link name="${frame_prefix}_inertial_link">
       <inertial>
           <origin xyz="0.0 0.0 0.0" />
@@ -215,10 +51,5 @@
       </inertial>
   </link>
-  <joint name="${frame_prefix}_inertial_joint" type="fixed">
-      <origin xyz="0 0 0" rpy="0 0 0" />
-      <parent link="${frame_prefix}_base_link" />
-      <child link="${frame_prefix}_inertial_link" />
-  </joint>
-  <!-- Sensor and wheel macros: pass prefixed names so all internal links are unique -->
+  <!-- Sensors with reduced update rates -->
   <xacro:limo_laser parent_prefix="${frame_prefix}_base_link" frame_prefix="${frame_prefix}_laser">
       <origin xyz="0.103 0 -0.034" rpy="0 0 0"/>
@@ -230,4 +61,5 @@
       <origin xyz="0.0 0 -0.1" rpy="0 0 0"/>
   </xacro:limo_imu>
+  <!-- Wheels -->
   <xacro:limo_wheel parent_prefix="${frame_prefix}_base_link" wheel_prefix="${frame_prefix}_front_left" reflect="1">
       <origin xyz="${wheelbase/2} ${track/2} ${wheel_vertical_offset}" rpy="0 0  0" />
@@ -242,3 +74,147 @@
       <origin xyz="${-wheelbase/2} ${-track/2} ${wheel_vertical_offset}" rpy="${M_PI} 0 0" />
   </xacro:limo_wheel>
+  <!-- Simplified Laser Sensor (reduced samples and update rate) -->
+  <gazebo reference="${frame_prefix}_laser_link">
+    <sensor type="ray" name="${frame_prefix}_laser_sensor">
+      <pose>0 0 0 0 0 0</pose>
+      <visualize>false</visualize>
+      <update_rate>5</update_rate>
+      <ray>
+        <scan>
+          <horizontal>
+            <samples>360</samples>
+            <resolution>1</resolution>
+            <min_angle>-2.09439504</min_angle>
+            <max_angle>2.09439504</max_angle>
+          </horizontal>
+        </scan>
+        <range>
+          <min>0.05</min>
+          <max>8.0</max>
+          <resolution>0.02</resolution>
+        </range>
+        <noise>
+          <type>gaussian</type>
+          <mean>0.0</mean>
+          <stddev>0.01</stddev>
+        </noise>
+      </ray>
+      <plugin name="${frame_prefix}_laser_plugin" filename="libgazebo_ros_laser.so">
+        <topicName>${robot_namespace}/scan</topicName>
+        <frameName>${frame_prefix}_laser_link</frameName>
+      </plugin>
+    </sensor>
+  </gazebo>
+  <!-- Simplified Depth Camera (lower resolution and update rate) -->
+  <gazebo reference="${frame_prefix}_depth_camera_link">
+    <sensor name="${frame_prefix}_depth_camera_sensor" type="depth">
+      <pose>0.0 0.0 0.0 0.0 0.0 0.0</pose>
+      <always_on>true</always_on>
+      <visualize>false</visualize>
+      <update_rate>5.0</update_rate>
+      <camera name="head">
+        <horizontal_fov>1.3962634</horizontal_fov>
+        <image>
+          <width>320</width>
+          <height>240</height>
+          <format>R8G8B8</format>
+        </image>
+        <clip>
+          <near>0.02</near>
+          <far>300</far>
+        </clip>
+      </camera>
+      <plugin name="${frame_prefix}_depth_camera_plugin" filename="libgazebo_ros_openni_kinect.so">
+        <baseline>0.2</baseline>
+        <alwaysOn>true</alwaysOn>
+        <updateRate>5.0</updateRate>
+        <cameraName>camera_ir</cameraName>
+        <imageTopicName>${robot_namespace}/color/image_raw</imageTopicName>
+        <cameraInfoTopicName>${robot_namespace}/color/camera_info</cameraInfoTopicName>
+        <depthImageTopicName>${robot_namespace}/depth/image_raw</depthImageTopicName>
+        <depthImageCameraInfoTopicName>${robot_namespace}/depth/camera_info</depthImageCameraInfoTopicName>
+        <pointCloudTopicName>${robot_namespace}/depth/points</pointCloudTopicName>
+        <frameName>${frame_prefix}_depth_camera_link</frameName>
+        <pointCloudCutoff>0.5</pointCloudCutoff>
+        <pointCloudCutoffMax>3.0</pointCloudCutoffMax>
+      </plugin>
+    </sensor>
+  </gazebo>
+  <!-- IMU with reduced update rate -->
+  <gazebo reference="${frame_prefix}_imu_link">
+    <gravity>true</gravity>
+    <sensor name="${frame_prefix}_imu_sensor" type="imu">
+      <always_on>true</always_on>
+      <update_rate>50</update_rate>
+      <visualize>false</visualize>
+      <plugin filename="libgazebo_ros_imu_sensor.so" name="${frame_prefix}_imu_plugin">
+        <topicName>${robot_namespace}/imu</topicName>
+        <bodyName>${frame_prefix}_imu_link</bodyName>
+        <updateRateHZ>50.0</updateRateHZ>
+        <gaussianNoise>0.001</gaussianNoise>
+        <xyzOffset>0 0 0</xyzOffset>
+        <rpyOffset>0 0 0</rpyOffset>
+        <frameName>${frame_prefix}_imu_link</frameName>
+      </plugin>
+    </sensor>
+  </gazebo>
+  <!-- Optimized wheel contact parameters -->
+  <gazebo reference="${frame_prefix}_front_left_wheel">
+      <mu1>10</mu1>
+      <mu2>10</mu2>
+      <kp>10000000.0</kp>
+      <kd>1.0</kd>
+      <minDepth>0.01</minDepth>
+      <fdir1>1 0 0</fdir1>
+      <maxContacts>10</maxContacts>
+  </gazebo>
+  <gazebo reference="${frame_prefix}_front_right_wheel">
+      <mu1>10</mu1>
+      <mu2>10</mu2>
+      <kp>10000000.0</kp>
+      <kd>1.0</kd>
+      <minDepth>0.01</minDepth>
+      <fdir1>1 0 0</fdir1>
+      <maxContacts>10</maxContacts>
+  </gazebo>
+  <gazebo reference="${frame_prefix}_rear_left_wheel">
+      <mu1>10</mu1>
+      <mu2>10</mu2>
+      <kp>10000000.0</kp>
+      <kd>1.0</kd>
+      <minDepth>0.01</minDepth>
+      <fdir1>1 0 0</fdir1>
+      <maxContacts>10</maxContacts>
+  </gazebo>
+  <gazebo reference="${frame_prefix}_rear_right_wheel">
+      <mu1>10</mu1>
+      <mu2>10</mu2>
+      <kp>10000000.0</kp>
+      <kd>1.0</kd>
+      <minDepth>0.01</minDepth>
+      <fdir1>1 0 0</fdir1>
+      <maxContacts>10</maxContacts>
+  </gazebo>
+  <!-- Skid-steer drive plugin with optimized update rate -->
+  <gazebo>
+      <plugin name="four_diff_controller" filename="libgazebo_ros_skid_steer_drive.so">
+          <updateRate>50.0</updateRate>
+          <robotNamespace>/${robot_namespace}</robotNamespace>
+          <leftFrontJoint>${frame_prefix}_front_left_wheel</leftFrontJoint>
+          <rightFrontJoint>${frame_prefix}_front_right_wheel</rightFrontJoint>
+          <leftRearJoint>${frame_prefix}_rear_left_wheel</leftRearJoint>
+          <rightRearJoint>${frame_prefix}_rear_right_wheel</rightRearJoint>
+          <wheelSeparation>0.172</wheelSeparation>
+          <wheelDiameter>0.09</wheelDiameter>
+          <robotBaseFrame>${frame_prefix}_base_footprint</robotBaseFrame>
+          <commandTopic>/${robot_namespace}/cmd_vel</commandTopic>
+          <torque>50</torque>
+          <broadcastTF>true</broadcastTF>
+          <odometryTopic>/${robot_namespace}/odom</odometryTopic>
+          <odometryFrame>${frame_prefix}_odom</odometryFrame>
+          <covariance_x>0.000100</covariance_x>
+          <covariance_y>0.000100</covariance_y>
+          <covariance_yaw>0.010000</covariance_yaw>
+      </plugin>
+  </gazebo>
 </robot>
